File: Custom Mechanical Keyboard.kicad_pcb (KiCad board)
At the start: 2 copper layers, 3.6 x 3.2 mm, 274 parts, among them SW1 SW_SPST, SW10 SW_SPST, SW11 SW_SPST, SW12 SW_SPST, SW13 SW_SPST, SW14 SW_SPST, SW15 SW_SPST, SW16 SW_SPST, SW17 SW_SPST, SW18 SW_SPST, SW19 SW_SPST, SW2 SW_SPST, SW20 SW_SPST, SW21 SW_SPST, SW22 SW_SPST, SW23 SW_SPST, SW24 SW_SPST, SW25 SW_SPST, SW26 SW_SPST, SW27 SW_SPST, SW28 SW_SPST, SW29 SW_SPST, SW3 SW_SPST, SW30 SW_SPST, SW31 SW_SPST, SW32 SW_SPST, SW33 SW_SPST, SW34 SW_SPST, SW35 SW_SPST, SW36 SW_SPST, SW37 SW_SPST, SW38 SW_SPST, SW39 SW_SPST, SW4 SW_SPST, SW40 SW_SPST, SW41 SW_SPST, SW42 SW_SPST, SW43 SW_SPST, SW44 SW_SPST, SW45 SW_SPST, SW46 SW_SPST, SW47 SW_SPST, SW48 SW_SPST, SW49 SW_SPST, SW5 SW_SPST, SW50 SW_SPST, SW51 SW_SPST, SW52 SW_SPST, SW53 SW_SPST, SW54 SW_SPST, SW55 SW_SPST, SW56 SW_SPST, SW57 SW_SPST, SW58 SW_SPST, SW59 SW_SPST, SW6 SW_SPST, SW60 SW_SPST, SW61 SW_SPST, SW62 SW_SPST, SW63 SW_SPST, SW64 SW_SPST, SW65 SW_SPST, SW66 SW_SPST, SW67 SW_SPST, SW68 SW_SPST, SW69 SW_SPST, SW7 SW_SPST, SW70 SW_SPST, SW71 SW_SPST, SW72 SW_SPST, SW73 SW_SPST, SW74 SW_SPST, SW75 SW_SPST, SW76 SW_SPST, SW77 SW_SPST, SW78 SW_SPST, SW79 SW_SPST, SW8 SW_SPST, SW80 SW_SPST, SW81 SW_SPST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

Commit message: Changed MCU position, swapped screw-in stab mounts for stab cutouts for gateron lp stabilizers
Parts:
- added REF**: STAB_MX_5u, PCM_marbastlib-mx:STAB_MX_5u, F.Cu at (152.4, 133.3)
- added REF**: STAB_MX_LP_2u, Gateron_LP_Stabilizers:STAB_MX_LP_2u, F.Cu at (276.2, 114.3)
- added REF**: STAB_MX_LP_2u, Gateron_LP_Stabilizers:STAB_MX_LP_2u, F.Cu at (290.5, 95.2)
- added REF**: STAB_MX_LP_2u, Gateron_LP_Stabilizers:STAB_MX_LP_2u, F.Cu at (295.3, 57.1)
- added REF**: STAB_MX_LP_2u, Gateron_LP_Stabilizers:STAB_MX_LP_2u, F.Cu at (47.6, 114.3)
- LED1, LED10, LED11, LED12, LED13, LED14, LED15, LED16, LED17, LED18, LED19, LED2, LED20, LED21, LED22, LED23, LED24, LED25, LED26, LED27, LED28, LED29, LED3, LED30, LED31, LED32, LED33, LED34, LED35, LED36, LED37, LED38, LED39, LED4, LED40, LED41, LED42, LED43, LED44, LED45, LED46, LED47, LED48, LED49, LED5, LED50, LED51, LED52, LED53, LED54, LED55, LED56, LED57, LED58, LED59, LED6, LED60, LED61, LED62, LED63, LED64, LED65, LED66, LED67, LED68, LED69, LED7, LED70, LED71, LED72, LED73, LED74, LED75, LED76, LED77, LED78, LED79, LED8, LED80, LED81, LED82, LED83, LED84, LED9: value SK6812MINI -> SK6812MINI-E; footprint LED_SMD:LED_SK6812MINI-E_PLCC4_3.2x2.8mm_P1.5mm -> LED_SMD:LED_SK6812MINI-E_Reversed_PLCC4_3.2x2.8mm_P1.5mm
- U2: moved to B.Cu
- moved U1 179.3 mm to (27.9, 141.1), turned to 90 degrees
- moved A9_USB_VBUS1 178.6 mm to (15.4, 128.4), turned to -90 degrees
- moved A10_USB_ID1 176.1 mm to (15.4, 125.8), turned to -90 degrees
- moved A11_USB_DM1 173.8 mm to (15.4, 123.3), turned to -90 degrees
- moved A12_USB_DP1 171.4 mm to (15.5, 120.8), turned to -90 degrees
- moved B2_BOOT1 170.8 mm to (25.8, 131.0)
- moved U2 160.4 mm to (20.1, 84.9), turned to 180 degrees
- moved SOI8_SLCT1 155.6 mm to (25.8, 115.7)
- moved NRST1 144.4 mm to (25.9, 103.0)
- moved VBat1 134.1 mm to (27.8, 88.7)
- moved C12 13.7 mm to (160.1, 127.3)
- moved C4 0.93 mm to (179.2, 51.2)
- moved C3 0.90 mm to (184.4, 51.2)
- moved C7 0.88 mm to (194.0, 89.3)
- moved C8 0.88 mm to (188.7, 89.3)
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Connections:
- net Row10 renamed Col10
- net Row11 renamed Col11
- net Row12 renamed Col12
- net Row13 renamed Col13
- net Row14 renamed Col14
- net Row15 renamed Col15
- net Row6 renamed Col6
- net Row7 renamed Col7
- net Row8 renamed Col8
- net Row9 renamed Col9
- D1 pad 1: Col0 -> Row0
- D10 pad 1: Col0 -> Row0
- D11 pad 1: Col0 -> Row0
- D12 pad 1: Col0 -> Row0
- D13 pad 1: Col0 -> Row0
- D14 pad 1: Col0 -> Row0
- D15 pad 1: Col0 -> Row0
- D16 pad 1: Col0 -> Row0
- D17 pad 1: Col1 -> Row1
- D18 pad 1: Col1 -> Row1
- D19 pad 1: Col1 -> Row1
- D2 pad 1: Col0 -> Row0
- D20 pad 1: Col1 -> Row1
- D21 pad 1: Col1 -> Row1
- D22 pad 1: Col1 -> Row1
- D23 pad 1: Col1 -> Row1
- D24 pad 1: Col1 -> Row1
- D25 pad 1: Col1 -> Row1
- D26 pad 1: Col1 -> Row1
- D27 pad 1: Col1 -> Row1
- D28 pad 1: Col1 -> Row1
- D29 pad 1: Col1 -> Row1
- D3 pad 1: Col0 -> Row0
- D30 pad 1: Col1 -> Row1
- D31 pad 1: Col1 -> Row1
- D32 pad 1: Col2 -> Row2
- D33 pad 1: Col2 -> Row2
- D34 pad 1: Col2 -> Row2
- D35 pad 1: Col2 -> Row2
- D36 pad 1: Col2 -> Row2
- D37 pad 1: Col2 -> Row2
- D38 pad 1: Col2 -> Row2
- D39 pad 1: Col2 -> Row2
- D4 pad 1: Col0 -> Row0
- D40 pad 1: Col2 -> Row2
- D41 pad 1: Col2 -> Row2
- D42 pad 1: Col2 -> Row2
- D43 pad 1: Col2 -> Row2
- D44 pad 1: Col2 -> Row2
- D45 pad 1: Col2 -> Row2
- D46 pad 1: Col2 -> Row2
- D47 pad 1: Col3 -> Row3
- D48 pad 1: Col3 -> Row3
- D49 pad 1: Col3 -> Row3
- D5 pad 1: Col0 -> Row0
- D50 pad 1: Col3 -> Row3
- D51 pad 1: Col3 -> Row3
- D52 pad 1: Col3 -> Row3
- D53 pad 1: Col3 -> Row3
- D54 pad 1: Col3 -> Row3
- D55 pad 1: Col3 -> Row3
- D56 pad 1: Col3 -> Row3
- D57 pad 1: Col3 -> Row3
- D58 pad 1: Col3 -> Row3
- D59 pad 1: Col3 -> Row3
- D6 pad 1: Col0 -> Row0
- D60 pad 1: Col3 -> Row3
- D61 pad 1: Col4 -> Row4
- D62 pad 1: Col4 -> Row4
- D63 pad 1: Col4 -> Row4
- D64 pad 1: Col4 -> Row4
- D65 pad 1: Col4 -> Row4
- D66 pad 1: Col4 -> Row4
- D67 pad 1: Col4 -> Row4
- D68 pad 1: Col4 -> Row4
- D69 pad 1: Col4 -> Row4
- D7 pad 1: Col0 -> Row0
- D70 pad 1: Col4 -> Row4
- D71 pad 1: Col4 -> Row4
- D72 pad 1: Col4 -> Row4
- D73 pad 1: Col4 -> Row4
- D74 pad 1: Col4 -> Row4
- D75 pad 1: Col5 -> Row5
- D76 pad 1: Col5 -> Row5
- D77 pad 1: Col5 -> Row5
- D78 pad 1: Col5 -> Row5
- D79 pad 1: Col5 -> Row5
- D8 pad 1: Col0 -> Row0
- D80 pad 1: Col5 -> Row5
- D81 pad 1: Col5 -> Row5
- D82 pad 1: Col5 -> Row5
- D83 pad 1: Col5 -> Row5
- D84 pad 1: Col5 -> Row5
- D9 pad 1: Col0 -> Row0
- LED1 pad 1: Net-(LED1-DOUT) -> +5V
- LED1 pad 2: GND -> Net-(LED1-DOUT)
- LED1 pad 4: +5V -> GND
- LED10 pad 1: Net-(LED10-DOUT) -> +5V
- LED10 pad 2: GND -> Net-(LED10-DOUT)
- LED10 pad 4: +5V -> GND
- LED11 pad 1: Net-(LED11-DOUT) -> +5V
- LED11 pad 2: GND -> Net-(LED11-DOUT)
- LED11 pad 4: +5V -> GND
- LED12 pad 1: Net-(LED12-DOUT) -> +5V
- LED12 pad 2: GND -> Net-(LED12-DOUT)
- LED12 pad 4: +5V -> GND
- LED13 pad 1: Net-(LED13-DOUT) -> +5V
- LED13 pad 2: GND -> Net-(LED13-DOUT)
- LED13 pad 4: +5V -> GND
- LED14 pad 1: Net-(LED14-DOUT) -> +5V
- LED14 pad 2: GND -> Net-(LED14-DOUT)
- LED14 pad 4: +5V -> GND
- LED15 pad 1: Net-(LED15-DOUT) -> +5V
- LED15 pad 2: GND -> Net-(LED15-DOUT)
- LED15 pad 4: +5V -> GND
- LED16 pad 1: Net-(LED16-DOUT) -> +5V
- LED16 pad 2: GND -> Net-(LED16-DOUT)
- LED16 pad 4: +5V -> GND
- LED17 pad 1: Net-(LED17-DOUT) -> +5V
- LED17 pad 2: GND -> Net-(LED17-DOUT)
- LED17 pad 4: +5V -> GND
- LED18 pad 1: Net-(LED18-DOUT) -> +5V
- LED18 pad 2: GND -> Net-(LED18-DOUT)
- LED18 pad 4: +5V -> GND
- LED19 pad 1: Net-(LED19-DOUT) -> +5V
- LED19 pad 2: GND -> Net-(LED19-DOUT)
- LED19 pad 4: +5V -> GND
- LED2 pad 1: Net-(LED2-DOUT) -> +5V
- LED2 pad 2: GND -> Net-(LED2-DOUT)
- LED2 pad 4: +5V -> GND
- LED20 pad 1: Net-(LED20-DOUT) -> +5V
- LED20 pad 2: GND -> Net-(LED20-DOUT)
- LED20 pad 4: +5V -> GND
- LED21 pad 1: Net-(LED21-DOUT) -> +5V
- LED21 pad 2: GND -> Net-(LED21-DOUT)
- LED21 pad 4: +5V -> GND
- LED22 pad 1: Net-(LED22-DOUT) -> +5V
- LED22 pad 2: GND -> Net-(LED22-DOUT)
- LED22 pad 4: +5V -> GND
- LED23 pad 1: Net-(LED23-DOUT) -> +5V
- LED23 pad 2: GND -> Net-(LED23-DOUT)
- LED23 pad 4: +5V -> GND
- LED24 pad 1: Net-(LED24-DOUT) -> +5V
- LED24 pad 2: GND -> Net-(LED24-DOUT)
- LED24 pad 4: +5V -> GND
- LED25 pad 1: Net-(LED25-DOUT) -> +5V
- LED25 pad 2: GND -> Net-(LED25-DOUT)
- LED25 pad 4: +5V -> GND
- LED26 pad 1: Net-(LED26-DOUT) -> +5V
- LED26 pad 2: GND -> Net-(LED26-DOUT)
- LED26 pad 4: +5V -> GND
- LED27 pad 1: Net-(LED27-DOUT) -> +5V
- LED27 pad 2: GND -> Net-(LED27-DOUT)
- LED27 pad 4: +5V -> GND
- LED28 pad 1: Net-(LED28-DOUT) -> +5V
- LED28 pad 2: GND -> Net-(LED28-DOUT)
- LED28 pad 4: +5V -> GND
- LED29 pad 1: Net-(LED29-DOUT) -> +5V
- LED29 pad 2: GND -> Net-(LED29-DOUT)
- LED29 pad 4: +5V -> GND
- LED3 pad 1: Net-(LED3-DOUT) -> +5V
- LED3 pad 2: GND -> Net-(LED3-DOUT)
- LED3 pad 4: +5V -> GND
- LED30 pad 1: Net-(LED30-DOUT) -> +5V
- LED30 pad 2: GND -> Net-(LED30-DOUT)
- LED30 pad 4: +5V -> GND
- LED31 pad 1: Net-(LED31-DOUT) -> +5V
- LED31 pad 2: GND -> Net-(LED31-DOUT)
- LED31 pad 4: +5V -> GND
- LED32 pad 1: Net-(LED32-DOUT) -> +5V
- LED32 pad 2: GND -> Net-(LED32-DOUT)
- LED32 pad 4: +5V -> GND
- LED33 pad 1: Net-(LED33-DOUT) -> +5V
- LED33 pad 2: GND -> Net-(LED33-DOUT)
- LED33 pad 4: +5V -> GND
- LED34 pad 1: Net-(LED34-DOUT) -> +5V
- LED34 pad 2: GND -> Net-(LED34-DOUT)
- LED34 pad 4: +5V -> GND
- LED35 pad 1: Net-(LED35-DOUT) -> +5V
- LED35 pad 2: GND -> Net-(LED35-DOUT)
- LED35 pad 4: +5V -> GND
- LED36 pad 1: Net-(LED36-DOUT) -> +5V
- LED36 pad 2: GND -> Net-(LED36-DOUT)
- LED36 pad 4: +5V -> GND
- LED37 pad 1: Net-(LED37-DOUT) -> +5V
- LED37 pad 2: GND -> Net-(LED37-DOUT)
- LED37 pad 4: +5V -> GND
- LED38 pad 1: Net-(LED38-DOUT) -> +5V
- LED38 pad 2: GND -> Net-(LED38-DOUT)
- LED38 pad 4: +5V -> GND
- LED39 pad 1: Net-(LED39-DOUT) -> +5V
- LED39 pad 2: GND -> Net-(LED39-DOUT)
- LED39 pad 4: +5V -> GND
- LED4 pad 1: Net-(LED4-DOUT) -> +5V
- LED4 pad 2: GND -> Net-(LED4-DOUT)
- LED4 pad 4: +5V -> GND
- LED40 pad 1: Net-(LED40-DOUT) -> +5V
- LED40 pad 2: GND -> Net-(LED40-DOUT)
- LED40 pad 4: +5V -> GND
- LED41 pad 1: Net-(LED41-DOUT) -> +5V
- LED41 pad 2: GND -> Net-(LED41-DOUT)
- LED41 pad 4: +5V -> GND
- LED42 pad 1: Net-(LED42-DOUT) -> +5V
- LED42 pad 2: GND -> Net-(LED42-DOUT)
- LED42 pad 4: +5V -> GND
- LED43 pad 1: Net-(LED43-DOUT) -> +5V
- LED43 pad 2: GND -> Net-(LED43-DOUT)
- LED43 pad 4: +5V -> GND
- LED44 pad 1: Net-(LED44-DOUT) -> +5V
- LED44 pad 2: GND -> Net-(LED44-DOUT)
- LED44 pad 4: +5V -> GND
- LED45 pad 1: Net-(LED45-DOUT) -> +5V
- LED45 pad 2: GND -> Net-(LED45-DOUT)
- LED45 pad 4: +5V -> GND
- LED46 pad 1: Net-(LED46-DOUT) -> +5V
- LED46 pad 2: GND -> Net-(LED46-DOUT)
- LED46 pad 4: +5V -> GND
- LED47 pad 1: Net-(LED47-DOUT) -> +5V
- LED47 pad 2: GND -> Net-(LED47-DOUT)
- LED47 pad 4: +5V -> GND
- LED48 pad 1: Net-(LED48-DOUT) -> +5V
- LED48 pad 2: GND -> Net-(LED48-DOUT)
- LED48 pad 4: +5V -> GND
- LED49 pad 1: Net-(LED49-DOUT) -> +5V
- LED49 pad 2: GND -> Net-(LED49-DOUT)
- LED49 pad 4: +5V -> GND
- LED5 pad 1: Net-(LED5-DOUT) -> +5V
- LED5 pad 2: GND -> Net-(LED5-DOUT)
- LED5 pad 4: +5V -> GND
- LED50 pad 1: Net-(LED50-DOUT) -> +5V
- LED50 pad 2: GND -> Net-(LED50-DOUT)
- LED50 pad 4: +5V -> GND
- LED51 pad 1: Net-(LED51-DOUT) -> +5V
- LED51 pad 2: GND -> Net-(LED51-DOUT)
- LED51 pad 4: +5V -> GND
- LED52 pad 1: Net-(LED52-DOUT) -> +5V
- LED52 pad 2: GND -> Net-(LED52-DOUT)
- LED52 pad 4: +5V -> GND
- LED53 pad 1: Net-(LED53-DOUT) -> +5V
- LED53 pad 2: GND -> Net-(LED53-DOUT)
- LED53 pad 4: +5V -> GND
- LED54 pad 1: Net-(LED54-DOUT) -> +5V
- LED54 pad 2: GND -> Net-(LED54-DOUT)
- LED54 pad 4: +5V -> GND
- LED55 pad 1: Net-(LED55-DOUT) -> +5V
- LED55 pad 2: GND -> Net-(LED55-DOUT)
- LED55 pad 4: +5V -> GND
- LED56 pad 1: Net-(LED56-DOUT) -> +5V
- LED56 pad 2: GND -> Net-(LED56-DOUT)
- LED56 pad 4: +5V -> GND
- LED57 pad 1: Net-(LED57-DOUT) -> +5V
- LED57 pad 2: GND -> Net-(LED57-DOUT)
- LED57 pad 4: +5V -> GND
- LED58 pad 1: Net-(LED58-DOUT) -> +5V
- LED58 pad 2: GND -> Net-(LED58-DOUT)
- LED58 pad 4: +5V -> GND
- LED59 pad 1: Net-(LED59-DOUT) -> +5V
- LED59 pad 2: GND -> Net-(LED59-DOUT)
- LED59 pad 4: +5V -> GND
- LED6 pad 1: Net-(LED6-DOUT) -> +5V
- LED6 pad 2: GND -> Net-(LED6-DOUT)
- LED6 pad 4: +5V -> GND
- LED60 pad 1: Net-(LED60-DOUT) -> +5V
- LED60 pad 2: GND -> Net-(LED60-DOUT)
- LED60 pad 4: +5V -> GND
- LED61 pad 1: Net-(LED61-DOUT) -> +5V
- LED61 pad 2: GND -> Net-(LED61-DOUT)
- LED61 pad 4: +5V -> GND
- LED62 pad 1: Net-(LED62-DOUT) -> +5V
- LED62 pad 2: GND -> Net-(LED62-DOUT)
- LED62 pad 4: +5V -> GND
- LED63 pad 1: Net-(LED63-DOUT) -> +5V
- LED63 pad 2: GND -> Net-(LED63-DOUT)
- LED63 pad 4: +5V -> GND
- LED64 pad 1: Net-(LED64-DOUT) -> +5V
- LED64 pad 2: GND -> Net-(LED64-DOUT)
- LED64 pad 4: +5V -> GND
- LED65 pad 1: Net-(LED65-DOUT) -> +5V
- LED65 pad 2: GND -> Net-(LED65-DOUT)
- LED65 pad 4: +5V -> GND
- LED66 pad 1: Net-(LED66-DOUT) -> +5V
- LED66 pad 2: GND -> Net-(LED66-DOUT)
- LED66 pad 4: +5V -> GND
- LED67 pad 1: Net-(LED67-DOUT) -> +5V
- LED67 pad 2: GND -> Net-(LED67-DOUT)
- LED67 pad 4: +5V -> GND
- LED68 pad 1: Net-(LED68-DOUT) -> +5V
- LED68 pad 2: GND -> Net-(LED68-DOUT)
- LED68 pad 4: +5V -> GND
- LED69 pad 1: Net-(LED69-DOUT) -> +5V
- LED69 pad 2: GND -> Net-(LED69-DOUT)
- LED69 pad 4: +5V -> GND
- LED7 pad 1: Net-(LED7-DOUT) -> +5V
- LED7 pad 2: GND -> Net-(LED7-DOUT)
- LED7 pad 4: +5V -> GND
- LED70 pad 1: Net-(LED70-DOUT) -> +5V
- LED70 pad 2: GND -> Net-(LED70-DOUT)
- LED70 pad 4: +5V -> GND
- LED71 pad 1: Net-(LED71-DOUT) -> +5V
- LED71 pad 2: GND -> Net-(LED71-DOUT)
- LED71 pad 4: +5V -> GND
- LED72 pad 1: Net-(LED72-DOUT) -> +5V
- LED72 pad 2: GND -> Net-(LED72-DOUT)
- LED72 pad 4: +5V -> GND
- LED73 pad 1: Net-(LED73-DOUT) -> +5V
- LED73 pad 2: GND -> Net-(LED73-DOUT)
- LED73 pad 4: +5V -> GND
- LED74 pad 1: Net-(LED74-DOUT) -> +5V
- LED74 pad 2: GND -> Net-(LED74-DOUT)
- LED74 pad 4: +5V -> GND
- LED75 pad 1: Net-(LED75-DOUT) -> +5V
- LED75 pad 2: GND -> Net-(LED75-DOUT)
- LED75 pad 4: +5V -> GND
- LED76 pad 1: Net-(LED76-DOUT) -> +5V
- LED76 pad 2: GND -> Net-(LED76-DOUT)
- LED76 pad 4: +5V -> GND
- LED77 pad 1: Net-(LED77-DOUT) -> +5V
- LED77 pad 2: GND -> Net-(LED77-DOUT)
- LED77 pad 4: +5V -> GND
- LED78 pad 1: Net-(LED78-DOUT) -> +5V
- LED78 pad 2: GND -> Net-(LED78-DOUT)
- LED78 pad 4: +5V -> GND
- LED79 pad 1: Net-(LED79-DOUT) -> +5V
- LED79 pad 2: GND -> Net-(LED79-DOUT)
- LED79 pad 4: +5V -> GND
- LED8 pad 1: Net-(LED8-DOUT) -> +5V
- LED8 pad 2: GND -> Net-(LED8-DOUT)
- LED8 pad 4: +5V -> GND
- LED80 pad 1: Net-(LED80-DOUT) -> +5V
- LED80 pad 2: GND -> Net-(LED80-DOUT)
- LED80 pad 4: +5V -> GND
- LED81 pad 1: Net-(LED81-DOUT) -> +5V
- LED81 pad 2: GND -> Net-(LED81-DOUT)
- LED81 pad 4: +5V -> GND
- LED82 pad 1: Net-(LED82-DOUT) -> +5V
- LED82 pad 2: GND -> Net-(LED82-DOUT)
- LED82 pad 4: +5V -> GND
- LED83 pad 1: Net-(LED83-DOUT) -> +5V
- LED83 pad 2: GND -> Net-(LED83-DOUT)
- LED83 pad 4: +5V -> GND
- LED84 pad 1: unconnected-(LED84-DOUT-Pad1) -> +5V
- LED84 pad 2: GND -> unconnected-(LED84-DOUT-Pad2)
- LED84 pad 4: +5V -> GND
- LED9 pad 1: Net-(LED10-DIN) -> +5V
- LED9 pad 2: GND -> Net-(LED10-DIN)
- LED9 pad 4: +5V -> GND
- SW1 pad 1: Row0 -> Col0
- SW17 pad 1: Row0 -> Col0
- SW18 pad 1: Row1 -> Col1
- SW19 pad 1: Row2 -> Col2
- SW2 pad 1: Row1 -> Col1
- SW20 pad 1: Row3 -> Col3
- SW21 pad 1: Row4 -> Col4
- SW22 pad 1: Row5 -> Col5
- SW3 pad 1: Row2 -> Col2
- SW32 pad 1: Row0 -> Col0
- SW33 pad 1: Row1 -> Col1
- SW34 pad 1: Row2 -> Col2
- SW35 pad 1: Row3 -> Col3
- SW36 pad 1: Row4 -> Col4
- SW37 pad 1: Row5 -> Col5
- SW4 pad 1: Row3 -> Col3
- SW47 pad 1: Row0 -> Col0
- SW48 pad 1: Row1 -> Col1
- SW49 pad 1: Row2 -> Col2
- SW5 pad 1: Row4 -> Col4
- SW50 pad 1: Row3 -> Col3
- SW51 pad 1: Row4 -> Col4
- SW52 pad 1: Row5 -> Col5
- SW6 pad 1: Row5 -> Col5
- SW61 pad 1: Row0 -> Col0
- SW62 pad 1: Row1 -> Col1
- SW63 pad 1: Row2 -> Col2
- SW64 pad 1: Row3 -> Col3
- SW65 pad 1: Row4 -> Col4
- SW66 pad 1: Row5 -> Col5
- SW75 pad 1: Row0 -> Col0
- SW76 pad 1: Row1 -> Col1
- SW77 pad 1: Row2 -> Col2
- SW78 pad 1: Row5 -> Col5
- U1 pad 10: unconnected-(U1-A15-Pad10) -> Row2
- U1 pad 11: unconnected-(U1-B3-Pad11) -> Row3
- U1 pad 12: unconnected-(U1-B4-Pad12) -> Row4
- U1 pad 13: unconnected-(U1-B5-Pad13) -> Row5
- U1 pad 14: Row3 -> unconnected-(U1-B6-Pad14)
- U1 pad 15: Row2 -> unconnected-(U1-B7-Pad15)
- U1 pad 16: Row1 -> unconnected-(U1-B8-Pad16)
- U1 pad 17: Row0 -> unconnected-(U1-B9-Pad17)
- U1 pad 42: Row4 -> Row0
- U1 pad 43: Row5 -> Row1
- U1 pad 5: unconnected-(U1-A8-Pad5) -> CAPS
Routing:
- net Col0: track 383.1 -> 95.4 mm, vias 1 -> 0
- net Col1: track 359.2 -> 101.4 mm, vias 1 -> 0
- net Col2: track 353.7 -> 99.4 mm, vias 1 -> 0
- net Col5: track 350.3 -> 101.4 mm
- net Col3: track 318.0 -> 82.3 mm, vias 1 -> 0
- net LED: track 226.6 -> 0.00 mm, vias 1 -> 0
- net Col4: track 289.4 -> 82.3 mm
- net Row5: track 109.0 -> 311.4 mm
- net Row4: track 120.6 -> 296.5 mm, vias 0 -> 6
- net Row3: track 150.0 -> 295.3 mm, vias 0 -> 4
- net Col15: track 222.4 -> 95.2 mm
- net Row2: track 182.8 -> 302.6 mm
- net Col14: track 199.5 -> 95.0 mm
- net Row1: track 206.0 -> 298.3 mm
- net Col11: track 150.3 -> 59.3 mm, vias 2 -> 0
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Other:
- board size 3.6 x 3.2 mm -> 30.9 x 17 mm
