File: Custom Mechanical Keyboard.kicad_pcb (KiCad board)
At the start: 2 copper layers, 324 x 132.8 mm, 300 parts, among them J1 USB_C_Receptacle_USB2.0_16P, J2 Conn_01x04_Pin, J3 Conn_01x04_Pin, SW1 RotaryEncoder_Switch_MP, SW10 SW_SPST, SW11 SW_SPST, SW12 SW_SPST, SW13 SW_SPST, SW14 SW_SPST, SW15 SW_SPST, SW16 SW_SPST, SW17 SW_SPST, SW18 SW_SPST, SW19 SW_SPST, SW2 SW_SPST, SW20 SW_SPST, SW21 SW_SPST, SW22 SW_SPST, SW23 SW_SPST, SW24 SW_SPST, SW25 SW_SPST, SW26 SW_SPST, SW27 SW_SPST, SW28 SW_SPST, SW29 SW_SPST, SW3 SW_SPST, SW30 SW_SPST, SW31 SW_SPST, SW32 SW_SPST, SW33 SW_SPST, SW34 SW_SPST, SW35 SW_SPST, SW36 SW_SPST, SW37 SW_SPST, SW38 SW_SPST, SW39 SW_SPST, SW4 SW_SPST, SW40 SW_SPST, SW41 SW_SPST, SW42 SW_SPST, SW43 SW_SPST, SW44 SW_SPST, SW45 SW_SPST, SW46 SW_SPST, SW47 SW_SPST, SW48 SW_SPST, SW49 SW_SPST, SW5 SW_SPST, SW50 SW_SPST, SW51 SW_SPST, SW52 SW_SPST, SW53 SW_SPST, SW54 SW_SPST, SW55 SW_SPST, SW56 SW_SPST, SW57 SW_SPST, SW58 SW_SPST, SW59 SW_SPST, SW6 SW_SPST, SW60 SW_SPST, SW61 SW_SPST, SW62 SW_SPST, SW63 SW_SPST, SW64 SW_SPST, SW65 SW_SPST, SW66 SW_SPST, SW67 SW_SPST, SW68 SW_SPST, SW69 SW_SPST, SW7 SW_SPST, SW70 SW_SPST, SW71 SW_SPST, SW72 SW_SPST, SW73 SW_SPST, SW74 SW_SPST, SW75 SW_SPST, SW76 SW_SPST, SW77 SW_SPST, SW78 SW_SPST, SW79 SW_SPST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

Commit message: Fixed matrix LED wiring, shifted LED 0.2mm closer to switch. Changed capslock LED to addressable LED connected to matrix LED array.
Parts:
- removed CAPS1: LED, Keyboard_Parts_Footprint:LED_3020_REFLOW
- added ?: , , F.Cu at (352.4, 57.1)
- added ?: , , F.Cu at (161.9, 57.1)
- added ?: , , F.Cu at (352.4, 152.4)
- added ?: , , F.Cu at (190.5, 95.2)
- added ?: , , F.Cu at (247.7, 95.2)
- added ?: , , F.Cu at (292.9, 152.4)
- added ?: , , F.Cu at (90.5, 114.3)
- added ?: , , F.Cu at (304.8, 95.2)
- added ?: , , F.Cu at (88.1, 152.4)
- added ?: , , F.Cu at (304.8, 114.3)
- added ?: , , F.Cu at (257.2, 57.1)
- added ?: , , F.Cu at (133.3, 114.3)
- added ?: , , F.Cu at (66.7, 57.1)
- added ?: , , F.Cu at (71.4, 95.2)
- added ?: , , F.Cu at (247.7, 114.3)
- added ?: , , F.Cu at (238.1, 152.4)
- added ?: , , F.Cu at (133.3, 95.2)
- added ?: , , F.Cu at (190.5, 114.3)
- added ?: , , F.Cu at (142.9, 152.4)
- added CAPS_LED1: SK6812MINI-E_Rev, LED_SMD:LED_SK6812MINI-E_PLCC4_3.2x2.8mm_P1.5mm_1, F.Cu at (71.2, 114.3)
- LED1: renamed from LED2; value SK6812MINI-E -> SK6812MINI-E_Rev
- LED10: renamed from LED11; value SK6812MINI-E -> SK6812MINI-E_Rev
- LED11: renamed from LED12; value SK6812MINI-E -> SK6812MINI-E_Rev
- LED12: renamed from LED13; value SK6812MINI-E -> SK6812MINI-E_Rev
- LED13: renamed from LED14; value SK6812MINI-E -> SK6812MINI-E_Rev
- LED14: renamed from LED15; value SK6812MINI-E -> SK6812MINI-E_Rev
- LED15: renamed from LED16; value SK6812MINI-E -> SK6812MINI-E_Rev
- LED16: renamed from LED17; value SK6812MINI-E -> SK6812MINI-E_Rev
- LED17: renamed from LED18; value SK6812MINI-E -> SK6812MINI-E_Rev
- LED18: renamed from LED19; value SK6812MINI-E -> SK6812MINI-E_Rev
- LED19: renamed from LED20; value SK6812MINI-E -> SK6812MINI-E_Rev
- LED2: renamed from LED3; value SK6812MINI-E -> SK6812MINI-E_Rev
- LED20: renamed from LED21; value SK6812MINI-E -> SK6812MINI-E_Rev
- LED21: renamed from LED22; value SK6812MINI-E -> SK6812MINI-E_Rev
- LED22: renamed from LED23; value SK6812MINI-E -> SK6812MINI-E_Rev
- LED23: renamed from LED24; value SK6812MINI-E -> SK6812MINI-E_Rev
- LED24: renamed from LED25; value SK6812MINI-E -> SK6812MINI-E_Rev
- LED25: renamed from LED26; value SK6812MINI-E -> SK6812MINI-E_Rev
- LED26: renamed from LED27; value SK6812MINI-E -> SK6812MINI-E_Rev
- LED27: renamed from LED28; value SK6812MINI-E -> SK6812MINI-E_Rev
- LED28: renamed from LED29; value SK6812MINI-E -> SK6812MINI-E_Rev
- LED29: renamed from LED30; value SK6812MINI-E -> SK6812MINI-E_Rev
- LED3: renamed from LED4; value SK6812MINI-E -> SK6812MINI-E_Rev
- LED30: renamed from LED31; value SK6812MINI-E -> SK6812MINI-E_Rev
- LED31: renamed from LED32; value SK6812MINI-E -> SK6812MINI-E_Rev
- LED32: renamed from LED33; value SK6812MINI-E -> SK6812MINI-E_Rev
- LED33: renamed from LED34; value SK6812MINI-E -> SK6812MINI-E_Rev
- LED34: renamed from LED35; value SK6812MINI-E -> SK6812MINI-E_Rev
- LED35: renamed from LED36; value SK6812MINI-E -> SK6812MINI-E_Rev
- LED36: renamed from LED37; value SK6812MINI-E -> SK6812MINI-E_Rev
- LED37: renamed from LED38; value SK6812MINI-E -> SK6812MINI-E_Rev
- LED38: renamed from LED39; value SK6812MINI-E -> SK6812MINI-E_Rev
- LED39: renamed from LED40; value SK6812MINI-E -> SK6812MINI-E_Rev
- LED4: renamed from LED5; value SK6812MINI-E -> SK6812MINI-E_Rev
- LED40: renamed from LED41; value SK6812MINI-E -> SK6812MINI-E_Rev
- LED41: renamed from LED42; value SK6812MINI-E -> SK6812MINI-E_Rev
- LED42: renamed from LED43; value SK6812MINI-E -> SK6812MINI-E_Rev
- LED43: renamed from LED44; value SK6812MINI-E -> SK6812MINI-E_Rev
- LED44: renamed from LED45; value SK6812MINI-E -> SK6812MINI-E_Rev
- LED45: renamed from LED46; value SK6812MINI-E -> SK6812MINI-E_Rev
- LED46: renamed from LED47; value SK6812MINI-E -> SK6812MINI-E_Rev
- LED47: renamed from LED48; value SK6812MINI-E -> SK6812MINI-E_Rev
- LED48: renamed from LED49; value SK6812MINI-E -> SK6812MINI-E_Rev
- LED49: renamed from LED50; value SK6812MINI-E -> SK6812MINI-E_Rev
- LED5: renamed from LED6; value SK6812MINI-E -> SK6812MINI-E_Rev
- LED50: renamed from LED51; value SK6812MINI-E -> SK6812MINI-E_Rev
- LED51: renamed from LED52; value SK6812MINI-E -> SK6812MINI-E_Rev
- LED52: renamed from LED53; value SK6812MINI-E -> SK6812MINI-E_Rev
- LED53: renamed from LED54; value SK6812MINI-E -> SK6812MINI-E_Rev
- LED54: renamed from LED55; value SK6812MINI-E -> SK6812MINI-E_Rev
- LED55: renamed from LED56; value SK6812MINI-E -> SK6812MINI-E_Rev
- LED56: renamed from LED57; value SK6812MINI-E -> SK6812MINI-E_Rev
- LED57: renamed from LED58; value SK6812MINI-E -> SK6812MINI-E_Rev
- LED58: renamed from LED59; value SK6812MINI-E -> SK6812MINI-E_Rev
- LED59: renamed from LED60; value SK6812MINI-E -> SK6812MINI-E_Rev
- LED6: renamed from LED7; value SK6812MINI-E -> SK6812MINI-E_Rev
- LED60: renamed from LED61; value SK6812MINI-E -> SK6812MINI-E_Rev
- LED61: renamed from LED62; value SK6812MINI-E -> SK6812MINI-E_Rev
- LED62: renamed from LED63; value SK6812MINI-E -> SK6812MINI-E_Rev
- LED63: renamed from LED64; value SK6812MINI-E -> SK6812MINI-E_Rev
- LED64: renamed from LED65; value SK6812MINI-E -> SK6812MINI-E_Rev
- LED65: renamed from LED66; value SK6812MINI-E -> SK6812MINI-E_Rev
- LED66: renamed from LED67; value SK6812MINI-E -> SK6812MINI-E_Rev
- LED67: renamed from LED68; value SK6812MINI-E -> SK6812MINI-E_Rev
- LED68: renamed from LED69; value SK6812MINI-E -> SK6812MINI-E_Rev
- LED69: renamed from LED70; value SK6812MINI-E -> SK6812MINI-E_Rev
- LED7: renamed from LED8; value SK6812MINI-E -> SK6812MINI-E_Rev
- LED70: renamed from LED71; value SK6812MINI-E -> SK6812MINI-E_Rev
- LED71: renamed from LED72; value SK6812MINI-E -> SK6812MINI-E_Rev
- LED72: renamed from LED73; value SK6812MINI-E -> SK6812MINI-E_Rev
- LED73: renamed from LED74; value SK6812MINI-E -> SK6812MINI-E_Rev
- LED74: renamed from LED75; value SK6812MINI-E -> SK6812MINI-E_Rev
- LED75: renamed from LED76; value SK6812MINI-E -> SK6812MINI-E_Rev
- LED76: renamed from LED77; value SK6812MINI-E -> SK6812MINI-E_Rev
- LED77: renamed from LED78; value SK6812MINI-E -> SK6812MINI-E_Rev
- LED78: renamed from LED79; value SK6812MINI-E -> SK6812MINI-E_Rev
- LED79: renamed from LED80; value SK6812MINI-E -> SK6812MINI-E_Rev
- LED8: renamed from LED9; value SK6812MINI-E -> SK6812MINI-E_Rev
- LED80: renamed from LED81; value SK6812MINI-E -> SK6812MINI-E_Rev
- LED81: renamed from LED82; value SK6812MINI-E -> SK6812MINI-E_Rev
- LED82: renamed from LED83; value SK6812MINI-E -> SK6812MINI-E_Rev
- LED83: renamed from LED84; value SK6812MINI-E -> SK6812MINI-E_Rev
- LED84: renamed from LED85; value SK6812MINI-E -> SK6812MINI-E_Rev
- LED9: renamed from LED10; value SK6812MINI-E -> SK6812MINI-E_Rev
- moved VBat1 1.65 mm to (66.1, 109.0)
- moved A12_USB_DP1 0.40 mm to (53.2, 139.7)
- moved A9_USB_VBUS1 0.40 mm to (53.2, 147.3)
- moved A10_USB_ID1 0.40 mm to (53.2, 144.8)
- moved A11_USB_DM1 0.40 mm to (53.2, 142.2)
- moved U1 0.39 mm to (66.1, 160.0)
- moved B2_BOOT1 0.39 mm to (63.9, 149.8)
- moved NRST1 0.39 mm to (63.9, 121.9)
- moved SOI8_SLCT1 0.39 mm to (63.9, 134.6)
- moved C1 0.22 mm to (204.0, 51.9)
- moved C4 0.21 mm to (89.8, 70.9)
- moved C10 0.20 mm to (108.7, 128.1)
- moved C11 0.20 mm to (248.8, 146.5)
- moved C12 0.20 mm to (96.8, 147.1)
- moved C6 0.20 mm to (223.1, 128.1)
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- renumbered D1 to CAPS_D1, SW1 to CAPS_SW1, D2 to D1, D11 to D10, D12 to D11, D13 to D12, D14 to D13, D15 to D14, D16 to D15, D17 to D16, D18 to D17, D19 to D18, D20 to D19, D3 to D2, D21 to D20, D22 to D21, D23 to D22, D24 to D23, D25 to D24, D26 to D25, D27 to D26, D28 to D27, D29 to D28, D30 to D29, D4 to D3, D31 to D30, D32 to D31, D33 to D32, D34 to D33, D35 to D34, D36 to D35, D37 to D36, D38 to D37, D39 to D38, D40 to D39, D5 to D4, D41 to D40, D42 to D41, D43 to D42, D44 to D43, D45 to D44, D46 to D45, D47 to D46, D48 to D47, D49 to D48, D50 to D49, D6 to D5, D51 to D50, D52 to D51, D53 to D52, D54 to D53, D55 to D54, D56 to D55, D57 to D56, D58 to D57, D59 to D58, D60 to D59, D7 to D6, D61 to D60, D62 to D61, D63 to D62, D64 to D63, D65 to D64, D66 to D65, D67 to D66, D68 to D67, D69 to D68, D70 to D69, D8 to D7, D71 to D70, D72 to D71, D73 to D72, D74 to D73, D75 to D74, D76 to D75, D77 to D76, D78 to D77, D79 to D78, D80 to D79, D9 to D8, D81 to D80, D82 to D81, D83 to D82, D84 to D83, D85 to D84, D10 to D9, D86 to ESD1, SW2 to SW1, SW11 to SW10, SW12 to SW11, SW13 to SW12, SW14 to SW13, SW15 to SW14, SW16 to SW15, SW17 to SW16, SW18 to SW17, SW19 to SW18, SW20 to SW19, SW3 to SW2, SW21 to SW20, SW22 to SW21, SW23 to SW22, SW24 to SW23, SW25 to SW24, SW26 to SW25, SW27 to SW26, SW28 to SW27, SW29 to SW28, SW30 to SW29, SW4 to SW3, SW31 to SW30, SW32 to SW31, SW33 to SW32, SW34 to SW33, SW35 to SW34, SW36 to SW35, SW37 to SW36, SW38 to SW37, SW39 to SW38, SW40 to SW39, SW5 to SW4, SW41 to SW40, SW42 to SW41, SW43 to SW42, SW44 to SW43, SW45 to SW44, SW46 to SW45, SW47 to SW46, SW48 to SW47, SW49 to SW48, SW50 to SW49, SW6 to SW5, SW51 to SW50, SW52 to SW51, SW53 to SW52, SW54 to SW53, SW55 to SW54, SW56 to SW55, SW57 to SW56, SW58 to SW57, SW59 to SW58, SW60 to SW59, SW7 to SW6, SW61 to SW60, SW62 to SW61, SW63 to SW62, SW64 to SW63, SW65 to SW64, SW66 to SW65, SW67 to SW66, SW68 to SW67, SW69 to SW68, SW70 to SW69, SW8 to SW7, SW71 to SW70, SW72 to SW71, SW73 to SW72, SW74 to SW73, SW75 to SW74, SW76 to SW75, SW77 to SW76, SW78 to SW77, SW79 to SW78, SW80 to SW79, SW9 to SW8, SW81 to SW80, SW82 to SW81, SW83 to SW82, SW84 to SW83, SW85 to SW84, SW10 to SW9
Connections:
- LED46 pad 2: Net-(LED47-DOUT) (its old number) -> Net-(CAPS_LED1-DIN)
- LED47 pad 3: Net-(LED47-DOUT) (its old number) -> Net-(CAPS_LED1-DOUT)
Routing:
- net Net-(CAPS_LED1-DIN): track 0.00 -> 320.1 mm, vias 0 -> 1
- net Net-(LED47-DOUT) (its old number): track 314.9 -> 0.00 mm
- net Net-(U1-A4): track 22.4 -> 2.21 mm
- net +5V: track 2077.3 -> 2096.4 mm, vias 7 -> 8
- net Net-(CAPS_LED1-DOUT): track 0.00 -> 11.2 mm, vias 0 -> 1
- net GND: track 2116.2 -> 2126.2 mm, vias 7 -> 8
- net Row5: track 483.4 -> 478.2 mm
- net EC_B: track 81.1 -> 77.7 mm
- net EC_A: track 82.9 -> 81.2 mm
- net Net-(U1-VBat): track 4.00 -> 2.35 mm
- net Col7: track 252.6 -> 254.2 mm
- net Col6: track 228.8 -> 230.4 mm
- net Col5: track 226.6 -> 228.2 mm
- net Col4: track 186.4 -> 188.0 mm
- net Col8: track 273.9 -> 275.4 mm
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