File: Custom Mechanical Keyboard.kicad_sch (KiCad schematic)
At the start: 274 parts, among them SW1 SW_SPST, SW10 SW_SPST, SW11 SW_SPST, SW12 SW_SPST, SW13 SW_SPST, SW14 SW_SPST, SW15 SW_SPST, SW16 SW_SPST, SW17 SW_SPST, SW18 SW_SPST, SW19 SW_SPST, SW2 SW_SPST, SW20 SW_SPST, SW21 SW_SPST, SW22 SW_SPST, SW23 SW_SPST, SW24 SW_SPST, SW25 SW_SPST, SW26 SW_SPST, SW27 SW_SPST, SW28 SW_SPST, SW29 SW_SPST, SW3 SW_SPST, SW30 SW_SPST, SW31 SW_SPST, SW32 SW_SPST, SW33 SW_SPST, SW34 SW_SPST, SW35 SW_SPST, SW36 SW_SPST, SW37 SW_SPST, SW38 SW_SPST, SW39 SW_SPST, SW4 SW_SPST, SW40 SW_SPST, SW41 SW_SPST, SW42 SW_SPST, SW43 SW_SPST, SW44 SW_SPST, SW45 SW_SPST, SW46 SW_SPST, SW47 SW_SPST, SW48 SW_SPST, SW49 SW_SPST, SW5 SW_SPST, SW50 SW_SPST, SW51 SW_SPST, SW52 SW_SPST, SW53 SW_SPST, SW54 SW_SPST, SW55 SW_SPST, SW56 SW_SPST, SW57 SW_SPST, SW58 SW_SPST, SW59 SW_SPST, SW6 SW_SPST, SW60 SW_SPST, SW61 SW_SPST, SW62 SW_SPST, SW63 SW_SPST, SW64 SW_SPST, SW65 SW_SPST, SW66 SW_SPST, SW67 SW_SPST, SW68 SW_SPST, SW69 SW_SPST, SW7 SW_SPST, SW70 SW_SPST, SW71 SW_SPST, SW72 SW_SPST, SW73 SW_SPST, SW74 SW_SPST, SW75 SW_SPST, SW76 SW_SPST, SW77 SW_SPST, SW78 SW_SPST, SW79 SW_SPST, SW8 SW_SPST, SW80 SW_SPST, SW81 SW_SPST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

Commit message: Changed MCU position, swapped screw-in stab mounts for stab cutouts for gateron lp stabilizers
Parts:
- LED1, LED10, LED11, LED12, LED13, LED14, LED15, LED16, LED17, LED18, LED19, LED2, LED20, LED21, LED22, LED23, LED24, LED25, LED26, LED27, LED28, LED29, LED3, LED30, LED31, LED32, LED33, LED34, LED35, LED36, LED37, LED38, LED39, LED4, LED40, LED41, LED42, LED43, LED44, LED45, LED46, LED47, LED48, LED49, LED5, LED50, LED51, LED52, LED53, LED54, LED55, LED56, LED57, LED58, LED59, LED6, LED60, LED61, LED62, LED63, LED64, LED65, LED66, LED67, LED68, LED69, LED7, LED70, LED71, LED72, LED73, LED74, LED75, LED76, LED77, LED78, LED79, LED8, LED80, LED81, LED82, LED83, LED84, LED9: value SK6812MINI -> SK6812MINI-E; footprint LED_SMD:LED_SK6812MINI-E_PLCC4_3.2x2.8mm_P1.5mm -> LED_SMD:LED_SK6812MINI-E_Reversed_PLCC4_3.2x2.8mm_P1.5mm; symbol LED:SK6812MINI -> LED_SMD:SK6812MINI-E
Connections:
- net +5V: now also LED1.1 (VDD), LED10.1 (VDD), LED11.1 (VDD), LED12.1 (VDD), LED13.1 (VDD), LED14.1 (VDD), LED15.1 (VDD), LED16.1 (VDD), LED17.1 (VDD), LED18.1 (VDD), LED19.1 (VDD), LED2.1 (VDD), LED20.1 (VDD), LED21.1 (VDD), LED22.1 (VDD), LED23.1 (VDD), LED24.1 (VDD), LED25.1 (VDD), LED26.1 (VDD), LED27.1 (VDD), LED28.1 (VDD), LED29.1 (VDD), LED3.1 (VDD), LED30.1 (VDD), LED31.1 (VDD), LED32.1 (VDD), LED33.1 (VDD), LED34.1 (VDD), LED35.1 (VDD), LED36.1 (VDD), LED37.1 (VDD), LED38.1 (VDD), LED39.1 (VDD), LED4.1 (VDD), LED40.1 (VDD), LED41.1 (VDD), LED42.1 (VDD), LED43.1 (VDD), LED44.1 (VDD), LED45.1 (VDD), LED46.1 (VDD), LED47.1 (VDD), LED48.1 (VDD), LED49.1 (VDD), LED5.1 (VDD), LED50.1 (VDD), LED51.1 (VDD), LED52.1 (VDD), LED53.1 (VDD), LED54.1 (VDD), LED55.1 (VDD), LED56.1 (VDD), LED57.1 (VDD), LED58.1 (VDD), LED59.1 (VDD), LED6.1 (VDD), LED60.1 (VDD), LED61.1 (VDD), LED62.1 (VDD), LED63.1 (VDD), LED64.1 (VDD), LED65.1 (VDD), LED66.1 (VDD), LED67.1 (VDD), LED68.1 (VDD), LED69.1 (VDD), LED7.1 (VDD), LED70.1 (VDD), LED71.1 (VDD), LED72.1 (VDD), LED73.1 (VDD), LED74.1 (VDD), LED75.1 (VDD), LED76.1 (VDD), LED77.1 (VDD), LED78.1 (VDD), LED79.1 (VDD), LED8.1 (VDD), LED80.1 (VDD), LED81.1 (VDD), LED82.1 (VDD), LED83.1 (VDD), LED84.1 (VDD), LED9.1 (VDD); no longer LED1.4 (VDD), LED10.4 (VDD), LED11.4 (VDD), LED12.4 (VDD), LED13.4 (VDD), LED14.4 (VDD), LED15.4 (VDD), LED16.4 (VDD), LED17.4 (VDD), LED18.4 (VDD), LED19.4 (VDD), LED2.4 (VDD), LED20.4 (VDD), LED21.4 (VDD), LED22.4 (VDD), LED23.4 (VDD), LED24.4 (VDD), LED25.4 (VDD), LED26.4 (VDD), LED27.4 (VDD), LED28.4 (VDD), LED29.4 (VDD), LED3.4 (VDD), LED30.4 (VDD), LED31.4 (VDD), LED32.4 (VDD), LED33.4 (VDD), LED34.4 (VDD), LED35.4 (VDD), LED36.4 (VDD), LED37.4 (VDD), LED38.4 (VDD), LED39.4 (VDD), LED4.4 (VDD), LED40.4 (VDD), LED41.4 (VDD), LED42.4 (VDD), LED43.4 (VDD), LED44.4 (VDD), LED45.4 (VDD), LED46.4 (VDD), LED47.4 (VDD), LED48.4 (VDD), LED49.4 (VDD), LED5.4 (VDD), LED50.4 (VDD), LED51.4 (VDD), LED52.4 (VDD), LED53.4 (VDD), LED54.4 (VDD), LED55.4 (VDD), LED56.4 (VDD), LED57.4 (VDD), LED58.4 (VDD), LED59.4 (VDD), LED6.4 (VDD), LED60.4 (VDD), LED61.4 (VDD), LED62.4 (VDD), LED63.4 (VDD), LED64.4 (VDD), LED65.4 (VDD), LED66.4 (VDD), LED67.4 (VDD), LED68.4 (VDD), LED69.4 (VDD), LED7.4 (VDD), LED70.4 (VDD), LED71.4 (VDD), LED72.4 (VDD), LED73.4 (VDD), LED74.4 (VDD), LED75.4 (VDD), LED76.4 (VDD), LED77.4 (VDD), LED78.4 (VDD), LED79.4 (VDD), LED8.4 (VDD), LED80.4 (VDD), LED81.4 (VDD), LED82.4 (VDD), LED83.4 (VDD), LED84.4 (VDD), LED9.4 (VDD)
- net Col0: now also SW1.1 (A), SW17.1 (A), SW32.1 (A), SW47.1 (A), SW61.1 (A), SW75.1 (A); no longer D1.1 (K), D10.1 (K), D11.1 (K), D12.1 (K), D13.1 (K), D14.1 (K), D15.1 (K), D16.1 (K), D2.1 (K), D3.1 (K), D4.1 (K), D5.1 (K), D6.1 (K), D7.1 (K), D8.1 (K), D9.1 (K)
- net Col1: now also SW18.1 (A), SW2.1 (A), SW33.1 (A), SW48.1 (A), SW62.1 (A), SW76.1 (A); no longer D17.1 (K), D18.1 (K), D19.1 (K), D20.1 (K), D21.1 (K), D22.1 (K), D23.1 (K), D24.1 (K), D25.1 (K), D26.1 (K), D27.1 (K), D28.1 (K), D29.1 (K), D30.1 (K), D31.1 (K)
- net Col2: now also SW19.1 (A), SW3.1 (A), SW34.1 (A), SW49.1 (A), SW63.1 (A), SW77.1 (A); no longer D32.1 (K), D33.1 (K), D34.1 (K), D35.1 (K), D36.1 (K), D37.1 (K), D38.1 (K), D39.1 (K), D40.1 (K), D41.1 (K), D42.1 (K), D43.1 (K), D44.1 (K), D45.1 (K), D46.1 (K)
- net Col3: now also SW20.1 (A), SW35.1 (A), SW4.1 (A), SW50.1 (A), SW64.1 (A); no longer D47.1 (K), D48.1 (K), D49.1 (K), D50.1 (K), D51.1 (K), D52.1 (K), D53.1 (K), D54.1 (K), D55.1 (K), D56.1 (K), D57.1 (K), D58.1 (K), D59.1 (K), D60.1 (K)
- net Col4: now also SW21.1 (A), SW36.1 (A), SW5.1 (A), SW51.1 (A), SW65.1 (A); no longer D61.1 (K), D62.1 (K), D63.1 (K), D64.1 (K), D65.1 (K), D66.1 (K), D67.1 (K), D68.1 (K), D69.1 (K), D70.1 (K), D71.1 (K), D72.1 (K), D73.1 (K), D74.1 (K)
- net Col5: now also SW22.1 (A), SW37.1 (A), SW52.1 (A), SW6.1 (A), SW66.1 (A), SW78.1 (A); no longer D75.1 (K), D76.1 (K), D77.1 (K), D78.1 (K), D79.1 (K), D80.1 (K), D81.1 (K), D82.1 (K), D83.1 (K), D84.1 (K)
- net GND: now also LED1.4 (GND), LED10.4 (GND), LED11.4 (GND), LED12.4 (GND), LED13.4 (GND), LED14.4 (GND), LED15.4 (GND), LED16.4 (GND), LED17.4 (GND), LED18.4 (GND), LED19.4 (GND), LED2.4 (GND), LED20.4 (GND), LED21.4 (GND), LED22.4 (GND), LED23.4 (GND), LED24.4 (GND), LED25.4 (GND), LED26.4 (GND), LED27.4 (GND), LED28.4 (GND), LED29.4 (GND), LED3.4 (GND), LED30.4 (GND), LED31.4 (GND), LED32.4 (GND), LED33.4 (GND), LED34.4 (GND), LED35.4 (GND), LED36.4 (GND), LED37.4 (GND), LED38.4 (GND), LED39.4 (GND), LED4.4 (GND), LED40.4 (GND), LED41.4 (GND), LED42.4 (GND), LED43.4 (GND), LED44.4 (GND), LED45.4 (GND), LED46.4 (GND), LED47.4 (GND), LED48.4 (GND), LED49.4 (GND), LED5.4 (GND), LED50.4 (GND), LED51.4 (GND), LED52.4 (GND), LED53.4 (GND), LED54.4 (GND), LED55.4 (GND), LED56.4 (GND), LED57.4 (GND), LED58.4 (GND), LED59.4 (GND), LED6.4 (GND), LED60.4 (GND), LED61.4 (GND), LED62.4 (GND), LED63.4 (GND), LED64.4 (GND), LED65.4 (GND), LED66.4 (GND), LED67.4 (GND), LED68.4 (GND), LED69.4 (GND), LED7.4 (GND), LED70.4 (GND), LED71.4 (GND), LED72.4 (GND), LED73.4 (GND), LED74.4 (GND), LED75.4 (GND), LED76.4 (GND), LED77.4 (GND), LED78.4 (GND), LED79.4 (GND), LED8.4 (GND), LED80.4 (GND), LED81.4 (GND), LED82.4 (GND), LED83.4 (GND), LED84.4 (GND), LED9.4 (GND); no longer LED1.2 (VSS), LED10.2 (VSS), LED11.2 (VSS), LED12.2 (VSS), LED13.2 (VSS), LED14.2 (VSS), LED15.2 (VSS), LED16.2 (VSS), LED17.2 (VSS), LED18.2 (VSS), LED19.2 (VSS), LED2.2 (VSS), LED20.2 (VSS), LED21.2 (VSS), LED22.2 (VSS), LED23.2 (VSS), LED24.2 (VSS), LED25.2 (VSS), LED26.2 (VSS), LED27.2 (VSS), LED28.2 (VSS), LED29.2 (VSS), LED3.2 (VSS), LED30.2 (VSS), LED31.2 (VSS), LED32.2 (VSS), LED33.2 (VSS), LED34.2 (VSS), LED35.2 (VSS), LED36.2 (VSS), LED37.2 (VSS), LED38.2 (VSS), LED39.2 (VSS), LED4.2 (VSS), LED40.2 (VSS), LED41.2 (VSS), LED42.2 (VSS), LED43.2 (VSS), LED44.2 (VSS), LED45.2 (VSS), LED46.2 (VSS), LED47.2 (VSS), LED48.2 (VSS), LED49.2 (VSS), LED5.2 (VSS), LED50.2 (VSS), LED51.2 (VSS), LED52.2 (VSS), LED53.2 (VSS), LED54.2 (VSS), LED55.2 (VSS), LED56.2 (VSS), LED57.2 (VSS), LED58.2 (VSS), LED59.2 (VSS), LED6.2 (VSS), LED60.2 (VSS), LED61.2 (VSS), LED62.2 (VSS), LED63.2 (VSS), LED64.2 (VSS), LED65.2 (VSS), LED66.2 (VSS), LED67.2 (VSS), LED68.2 (VSS), LED69.2 (VSS), LED7.2 (VSS), LED70.2 (VSS), LED71.2 (VSS), LED72.2 (VSS), LED73.2 (VSS), LED74.2 (VSS), LED75.2 (VSS), LED76.2 (VSS), LED77.2 (VSS), LED78.2 (VSS), LED79.2 (VSS), LED8.2 (VSS), LED80.2 (VSS), LED81.2 (VSS), LED82.2 (VSS), LED83.2 (VSS), LED84.2 (VSS), LED9.2 (VSS)
- net Row0: now also D1.1 (K), D10.1 (K), D11.1 (K), D12.1 (K), D13.1 (K), D14.1 (K), D15.1 (K), D16.1 (K), D2.1 (K), D3.1 (K), D4.1 (K), D5.1 (K), D6.1 (K), D7.1 (K), D8.1 (K), D9.1 (K), U1.42 (A13_DIO); no longer SW1.1 (A), SW17.1 (A), SW32.1 (A), SW47.1 (A), SW61.1 (A), SW75.1 (A), U1.17 (B9)
- net Row1: now also D17.1 (K), D18.1 (K), D19.1 (K), D20.1 (K), D21.1 (K), D22.1 (K), D23.1 (K), D24.1 (K), D25.1 (K), D26.1 (K), D27.1 (K), D28.1 (K), D29.1 (K), D30.1 (K), D31.1 (K), U1.43 (A14_SCK); no longer SW18.1 (A), SW2.1 (A), SW33.1 (A), SW48.1 (A), SW62.1 (A), SW76.1 (A), U1.16 (B8)
- net Row2: now also D32.1 (K), D33.1 (K), D34.1 (K), D35.1 (K), D36.1 (K), D37.1 (K), D38.1 (K), D39.1 (K), D40.1 (K), D41.1 (K), D42.1 (K), D43.1 (K), D44.1 (K), D45.1 (K), D46.1 (K), U1.10 (A15); no longer SW19.1 (A), SW3.1 (A), SW34.1 (A), SW49.1 (A), SW63.1 (A), SW77.1 (A), U1.15 (B7)
- net Row3: now also D47.1 (K), D48.1 (K), D49.1 (K), D50.1 (K), D51.1 (K), D52.1 (K), D53.1 (K), D54.1 (K), D55.1 (K), D56.1 (K), D57.1 (K), D58.1 (K), D59.1 (K), D60.1 (K), U1.11 (B3); no longer SW20.1 (A), SW35.1 (A), SW4.1 (A), SW50.1 (A), SW64.1 (A), U1.14 (B6)
- net Row4: now also D61.1 (K), D62.1 (K), D63.1 (K), D64.1 (K), D65.1 (K), D66.1 (K), D67.1 (K), D68.1 (K), D69.1 (K), D70.1 (K), D71.1 (K), D72.1 (K), D73.1 (K), D74.1 (K), U1.12 (B4); no longer SW21.1 (A), SW36.1 (A), SW5.1 (A), SW51.1 (A), SW65.1 (A), U1.42 (A13_DIO)
- net Row5: now also D75.1 (K), D76.1 (K), D77.1 (K), D78.1 (K), D79.1 (K), D80.1 (K), D81.1 (K), D82.1 (K), D83.1 (K), D84.1 (K), U1.13 (B5); no longer SW22.1 (A), SW37.1 (A), SW52.1 (A), SW6.1 (A), SW66.1 (A), SW78.1 (A), U1.43 (A14_SCK)
- net at LED62.3 (DIN): now also LED61.2 (DOUT); no longer LED61.1 (DOUT)
- net at LED61.3 (DIN): now also LED60.2 (DOUT); no longer LED60.1 (DOUT)
- net at LED57.3 (DIN): now also LED56.2 (DOUT); no longer LED56.1 (DOUT)
- net at LED56.3 (DIN): now also LED55.2 (DOUT); no longer LED55.1 (DOUT)
- net at LED44.3 (DIN): now also LED43.2 (DOUT); no longer LED43.1 (DOUT)
- net at LED43.3 (DIN): now also LED42.2 (DOUT); no longer LED42.1 (DOUT)
- net at LED54.3 (DIN): now also LED53.2 (DOUT); no longer LED53.1 (DOUT)
- net at LED53.3 (DIN): now also LED52.2 (DOUT); no longer LED52.1 (DOUT)
- net at LED15.3 (DIN): now also LED14.2 (DOUT); no longer LED14.1 (DOUT)
- net at LED14.3 (DIN): now also LED13.2 (DOUT); no longer LED13.1 (DOUT)
- net at LED84.3 (DIN): now also LED83.2 (DOUT); no longer LED83.1 (DOUT)
- net at LED83.3 (DIN): now also LED82.2 (DOUT); no longer LED82.1 (DOUT)
- net at LED42.3 (DIN): now also LED41.2 (DOUT); no longer LED41.1 (DOUT)
- net at LED41.3 (DIN): now also LED40.2 (DOUT); no longer LED40.1 (DOUT)
- net at LED78.3 (DIN): now also LED77.2 (DOUT); no longer LED77.1 (DOUT)
- net at LED77.3 (DIN): now also LED76.2 (DOUT); no longer LED76.1 (DOUT)
- net at LED32.3 (DIN): now also LED31.2 (DOUT); no longer LED31.1 (DOUT)
- net at LED31.3 (DIN): now also LED30.2 (DOUT); no longer LED30.1 (DOUT)
- net at LED75.3 (DIN): now also LED74.2 (DOUT); no longer LED74.1 (DOUT)
- net at LED74.3 (DIN): now also LED73.2 (DOUT); no longer LED73.1 (DOUT)
- net at LED19.3 (DIN): now also LED18.2 (DOUT); no longer LED18.1 (DOUT)
- net at LED18.3 (DIN): now also LED17.2 (DOUT); no longer LED17.1 (DOUT)
- net at LED25.3 (DIN): now also LED24.2 (DOUT); no longer LED24.1 (DOUT)
- net at LED24.3 (DIN): now also LED23.2 (DOUT); no longer LED23.1 (DOUT)
- net at LED28.3 (DIN): now also LED27.2 (DOUT); no longer LED27.1 (DOUT)
- net at LED27.3 (DIN): now also LED26.2 (DOUT); no longer LED26.1 (DOUT)
- net at LED30.3 (DIN): now also LED29.2 (DOUT); no longer LED29.1 (DOUT)
- net at LED29.3 (DIN): now also LED28.2 (DOUT); no longer LED28.1 (DOUT)
- net at LED59.3 (DIN): now also LED58.2 (DOUT); no longer LED58.1 (DOUT)
- net at LED58.3 (DIN): now also LED57.2 (DOUT); no longer LED57.1 (DOUT)
- net at LED82.3 (DIN): now also LED81.2 (DOUT); no longer LED81.1 (DOUT)
- net at LED40.3 (DIN): now also LED39.2 (DOUT); no longer LED39.1 (DOUT)
- net at LED39.3 (DIN): now also LED38.2 (DOUT); no longer LED38.1 (DOUT)
- net at LED76.3 (DIN): now also LED75.2 (DOUT); no longer LED75.1 (DOUT)
- net at LED5.3 (DIN): now also LED4.2 (DOUT); no longer LED4.1 (DOUT)
- net at LED4.3 (DIN): now also LED3.2 (DOUT); no longer LED3.1 (DOUT)
- net at LED49.3 (DIN): now also LED48.2 (DOUT); no longer LED48.1 (DOUT)
- net at LED48.3 (DIN): now also LED47.2 (DOUT); no longer LED47.1 (DOUT)
- net at LED35.3 (DIN): now also LED34.2 (DOUT); no longer LED34.1 (DOUT)
- net at LED34.3 (DIN): now also LED33.2 (DOUT); no longer LED33.1 (DOUT)
- net at LED64.3 (DIN): now also LED63.2 (DOUT); no longer LED63.1 (DOUT)
- net at LED63.3 (DIN): now also LED62.2 (DOUT); no longer LED62.1 (DOUT)
- net at LED71.3 (DIN): now also LED70.2 (DOUT); no longer LED70.1 (DOUT)
- net at LED70.3 (DIN): now also LED69.2 (DOUT); no longer LED69.1 (DOUT)
- net at LED33.3 (DIN): now also LED32.2 (DOUT); no longer LED32.1 (DOUT)
- net at LED9.3 (DIN): now also LED8.2 (DOUT); no longer LED8.1 (DOUT)
- net at LED8.3 (DIN): now also LED7.2 (DOUT); no longer LED7.1 (DOUT)
- net at LED45.3 (DIN): now also LED44.2 (DOUT); no longer LED44.1 (DOUT)
- net at LED12.3 (DIN): now also LED11.2 (DOUT); no longer LED11.1 (DOUT)
- net at LED11.3 (DIN): now also LED10.2 (DOUT); no longer LED10.1 (DOUT)
- net at LED17.3 (DIN): now also LED16.2 (DOUT); no longer LED16.1 (DOUT)
- net at LED16.3 (DIN): now also LED15.2 (DOUT); no longer LED15.1 (DOUT)
- net at LED68.3 (DIN): now also LED67.2 (DOUT); no longer LED67.1 (DOUT)
- net at LED67.3 (DIN): now also LED66.2 (DOUT); no longer LED66.1 (DOUT)
- net at LED80.3 (DIN): now also LED79.2 (DOUT); no longer LED79.1 (DOUT)
- net at LED79.3 (DIN): now also LED78.2 (DOUT); no longer LED78.1 (DOUT)
- net at LED37.3 (DIN): now also LED36.2 (DOUT); no longer LED36.1 (DOUT)
- net at LED36.3 (DIN): now also LED35.2 (DOUT); no longer LED35.1 (DOUT)
- net at LED6.3 (DIN): now also LED5.2 (DOUT); no longer LED5.1 (DOUT)
- net at LED38.3 (DIN): now also LED37.2 (DOUT); no longer LED37.1 (DOUT)
- net at LED73.3 (DIN): now also LED72.2 (DOUT); no longer LED72.1 (DOUT)
- net at LED60.3 (DIN): now also LED59.2 (DOUT); no longer LED59.1 (DOUT)
- net at LED69.3 (DIN): now also LED68.2 (DOUT); no longer LED68.1 (DOUT)
- net at LED65.3 (DIN): now also LED64.2 (DOUT); no longer LED64.1 (DOUT)
- net at LED13.3 (DIN): now also LED12.2 (DOUT); no longer LED12.1 (DOUT)
- net at LED23.3 (DIN): now also LED22.2 (DOUT); no longer LED22.1 (DOUT)
- net at LED47.3 (DIN): now also LED46.2 (DOUT); no longer LED46.1 (DOUT)
- net at LED52.3 (DIN): now also LED51.2 (DOUT); no longer LED51.1 (DOUT)
- net at LED66.3 (DIN): now also LED65.2 (DOUT); no longer LED65.1 (DOUT)
- net at LED22.3 (DIN): now also LED21.2 (DOUT); no longer LED21.1 (DOUT)
- net at LED21.3 (DIN): now also LED20.2 (DOUT); no longer LED20.1 (DOUT)
- net at LED72.3 (DIN): now also LED71.2 (DOUT); no longer LED71.1 (DOUT)
- net at LED46.3 (DIN): now also LED45.2 (DOUT); no longer LED45.1 (DOUT)
- net at LED50.3 (DIN): now also LED49.2 (DOUT); no longer LED49.1 (DOUT)
- net at LED20.3 (DIN): now also LED19.2 (DOUT); no longer LED19.1 (DOUT)
- net at LED7.3 (DIN): now also LED6.2 (DOUT); no longer LED6.1 (DOUT)
- net at LED10.3 (DIN): now also LED9.2 (DOUT); no longer LED9.1 (DOUT)
- net at LED55.3 (DIN): now also LED54.2 (DOUT); no longer LED54.1 (DOUT)
- net CAPS: now reaches U1.5 (A8)
- net at LED51.3 (DIN): now also LED50.2 (DOUT); no longer LED50.1 (DOUT)
- net at LED3.3 (DIN): now also LED2.2 (DOUT); no longer LED2.1 (DOUT)
- net at LED2.3 (DIN): now also LED1.2 (DOUT); no longer LED1.1 (DOUT)
- net at LED26.3 (DIN): now also LED25.2 (DOUT); no longer LED25.1 (DOUT)
- net at LED81.3 (DIN): now also LED80.2 (DOUT); no longer LED80.1 (DOUT)
- net Row10 renamed Col10
- net Row11 renamed Col11
- net Row12 renamed Col12
- net Row13 renamed Col13
- net Row14 renamed Col14
- net Row15 renamed Col15
- net Row6 renamed Col6
- net Row7 renamed Col7
- net Row8 renamed Col8
- net Row9 renamed Col9

Commit message: Updated wiring, board size, and added rotary encoder and usbc recepticle with esd protection as separate board
Parts:
- removed U2: TXS0102DCU, Package_SO:VSSOP-8_2.3x2mm_P0.5mm, symbol Logic_LevelTranslator:TXS0102DCU
- added CAPS1: LED, Keyboard_Parts_Footprint:LED_3020_REFLOW, symbol keyboard_parts:LED
- added D1: D, Keyboard_Parts_Footprint:D_SOD123, symbol Device:D
- added D86: SP0503BAHT, Package_TO_SOT_SMD:SOT-143, symbol Power_Protection:SP0503BAHT
- added J1: USB_C_Receptacle_USB2.0_16P, Connector_USB:USB_C_Receptacle_G-Switch_GT-USB-7010ASV, symbol Connector:USB_C_Receptacle_USB2.0_16P
- added J2, J3: Conn_01x04_Pin, Connector_JST:JST_PH_B4B-PH-K_1x04_P2.00mm_Vertical, symbol Connector:Conn_01x04_Pin
- added R1, R2: 5.1k, Resistor_SMD:R_1206_3216Metric_Pad1.30x1.75mm_HandSolder, symbol Device:R
- added SW1: RotaryEncoder_Switch_MP, Rotary_Encoder:RotaryEncoder_Alps_EC12E-Switch_Vertical_H20mm, symbol Device:RotaryEncoder_Switch_MP
- added U2: TXS0101DBV, Package_TO_SOT_SMD:SOT-23-6, symbol Logic_LevelTranslator:TXS0101DBV
- renumbered D9 to D10, D10 to D11, D11 to D12, D12 to D13, D13 to D14, D14 to D15, D15 to D16, D16 to D17, D17 to D18, D18 to D19, D1 to D2, D19 to D20, D20 to D21, D21 to D22, D22 to D23, D23 to D24, D24 to D25, D25 to D26, D26 to D27, D27 to D28, D28 to D29, D2 to D3, D29 to D30, D30 to D31, D31 to D32, D32 to D33, D33 to D34, D34 to D35, D35 to D36, D36 to D37, D37 to D38, D38 to D39, D3 to D4, D39 to D40, D40 to D41, D41 to D42, D42 to D43, D43 to D44, D44 to D45, D45 to D46, D46 to D47, D47 to D48, D48 to D49, D4 to D5, D49 to D50, D50 to D51, D51 to D52, D52 to D53, D53 to D54, D54 to D55, D55 to D56, D56 to D57, D57 to D58, D58 to D59, D5 to D6, D59 to D60, D60 to D61, D61 to D62, D62 to D63, D63 to D64, D64 to D65, D65 to D66, D66 to D67, D67 to D68, D68 to D69, D6 to D7, D69 to D70, D70 to D71, D71 to D72, D72 to D73, D73 to D74, D74 to D75, D75 to D76, D76 to D77, D77 to D78, D78 to D79, D7 to D8, D79 to D80, D80 to D81, D81 to D82, D82 to D83, D83 to D84, D84 to D85, D8 to D9, LED9 to LED10, LED10 to LED11, LED11 to LED12, LED12 to LED13, LED13 to LED14, LED14 to LED15, LED15 to LED16, LED16 to LED17, LED17 to LED18, LED18 to LED19, LED1 to LED2, LED19 to LED20, LED20 to LED21, LED21 to LED22, LED22 to LED23, LED23 to LED24, LED24 to LED25, LED25 to LED26, LED26 to LED27, LED27 to LED28, LED28 to LED29, LED2 to LED3, LED29 to LED30, LED30 to LED31, LED31 to LED32, LED32 to LED33, LED33 to LED34, LED34 to LED35, LED35 to LED36, LED36 to LED37, LED37 to LED38, LED38 to LED39, LED3 to LED4, LED39 to LED40, LED40 to LED41, LED41 to LED42, LED42 to LED43, LED43 to LED44, LED44 to LED45, LED45 to LED46, LED46 to LED47, LED47 to LED48, LED48 to LED49, LED4 to LED5, LED49 to LED50, LED50 to LED51, LED51 to LED52, LED52 to LED53, LED53 to LED54, LED54 to LED55, LED55 to LED56, LED56 to LED57, LED57 to LED58, LED58 to LED59, LED5 to LED6, LED59 to LED60, LED60 to LED61, LED61 to LED62, LED62 to LED63, LED63 to LED64, LED64 to LED65, LED65 to LED66, LED66 to LED67, LED67 to LED68, LED68 to LED69, LED6 to LED7, LED69 to LED70, LED70 to LED71, LED71 to LED72, LED72 to LED73, LED73 to LED74, LED74 to LED75, LED75 to LED76, LED76 to LED77, LED77 to LED78, LED78 to LED79, LED7 to LED8, LED79 to LED80, LED80 to LED81, LED81 to LED82, LED82 to LED83, LED83 to LED84, LED84 to LED85, LED8 to LED9, SW9 to SW10, SW10 to SW11, SW11 to SW12, SW12 to SW13, SW13 to SW14, SW14 to SW15, SW15 to SW16, SW16 to SW17, SW17 to SW18, SW18 to SW19, SW1 to SW2, SW19 to SW20, SW20 to SW21, SW21 to SW22, SW22 to SW23, SW23 to SW24, SW24 to SW25, SW25 to SW26, SW26 to SW27, SW27 to SW28, SW28 to SW29, SW2 to SW3, SW29 to SW30, SW30 to SW31, SW31 to SW32, SW32 to SW33, SW33 to SW34, SW34 to SW35, SW35 to SW36, SW36 to SW37, SW37 to SW38, SW38 to SW39, SW3 to SW4, SW39 to SW40, SW40 to SW41, SW41 to SW42, SW42 to SW43, SW43 to SW44, SW44 to SW45, SW45 to SW46, SW46 to SW47, SW47 to SW48, SW48 to SW49, SW4 to SW5, SW49 to SW50, SW50 to SW51, SW51 to SW52, SW52 to SW53, SW53 to SW54, SW54 to SW55, SW55 to SW56, SW56 to SW57, SW57 to SW58, SW58 to SW59, SW5 to SW6, SW59 to SW60, SW60 to SW61, SW61 to SW62, SW62 to SW63, SW63 to SW64, SW64 to SW65, SW65 to SW66, SW66 to SW67, SW67 to SW68, SW68 to SW69, SW6 to SW7, SW69 to SW70, SW70 to SW71, SW71 to SW72, SW72 to SW73, SW73 to SW74, SW74 to SW75, SW75 to SW76, SW76 to SW77, SW77 to SW78, SW78 to SW79, SW7 to SW8, SW79 to SW80, SW80 to SW81, SW81 to SW82, SW82 to SW83, SW83 to SW84, SW84 to SW85, SW8 to SW9
Connections:
- net CAPS is gone; now on net Col2: U1.5 (A8)
- net +3.3V: now also U2.1 (V_{CCA}), U2.5 (OE)
- net +5V: now also U2.6 (V_{CCB})
- net Col0: now also U1.28 (A2); no longer U1.22 (C13)
- net Col1: now also U1.29 (A3); no longer U1.23 (C14)
- net Col10: now also U1.11 (B3); no longer U1.35 (B1)
- net Col11: now also U1.10 (A15); no longer U1.37 (B10)
- net Col12: now also U1.16 (B8); no longer U1.1 (B12)
- net Col13: now also U1.15 (B7); no longer U1.2 (B13)
- net Col14: now also U1.14 (B6); no longer U1.3 (B14)
- net Col15: now also U1.13 (B5); no longer U1.4 (B15)
- net Col2: no longer U1.24 (C15)
- net Col3: now also U1.4 (B15), SW1.S1; no longer U1.26 (A0)
- net Col4: now also U1.22 (C13); no longer U1.27 (A1)
- net Col5: now also U1.23 (C14); no longer U1.28 (A2)
- net Col6: now also U1.24 (C15); no longer U1.31 (A5)
- net Col7: now also U1.26 (A0); no longer U1.32 (A6)
- net Col8: now also U1.27 (A1); no longer U1.33 (A7)
- net Col9: now also U1.12 (B4); no longer U1.34 (B0)
- net GND: now also CAPS1.1 (K), J3.1 (Pin_1), SW1.C, SW1.MP, U2.2 (GND)
- net Row2: now also U1.33 (A7); no longer U1.10 (A15)
- net Row3: now also U1.34 (B0); no longer U1.11 (B3)
- net Row4: now also U1.35 (B1); no longer U1.12 (B4)
- net Row5: now also U1.37 (B10), D1.1 (K); no longer U1.13 (B5)
- net USB_DM: now reaches A11_USB_DM1.1, U1.8 (A11_USBDM)
- net USB_DM: now also J3.3 (Pin_3)
- net USB_DP: now reaches A12_USB_DP1.1, U1.9 (A12_USBDP)
- net USB_DP: now also J3.2 (Pin_2)
- net USB_VBUS: now reaches A9_USB_VBUS1.1, U1.6 (A9_USBVB)
- net USB_VBUS: now also J3.4 (Pin_4)
- net at SOI8_SLCT1.1, U1.30 (A4): now also CAPS1.2 (A)
- net LED_3v3: now reaches U1.17 (B9)
- net LED_3v3: now also U2.3 (A)
- net LED renamed LED_5v
- net LED_5v: now also U2.4 (B)
- new net: J1.A5 (CC1), R2.1
- new net: J1.B5 (CC2), R1.1
- new net: D1.2 (A), SW1.S2
- new net DM: D86.3 (K), J1.A7 (D-), J1.B7 (D-), J2.3 (Pin_3)
- new net DP: D86.4 (K), J1.A6 (D+), J1.B6 (D+), J2.2 (Pin_2)
- new net EC_A: SW1.A, U1.32 (A6)
- new net EC_B: SW1.B, U1.31 (A5)
- new net USB_GND: D86.1 (A), J1.A1 (GND), J1.A12 (GND), J1.B1 (GND), J1.B12 (GND), J1.S1 (SHIELD), J2.1 (Pin_1), R1.2, R2.2
- new net VBUS: D86.2 (K), J1.A4 (VBUS), J1.A9 (VBUS), J1.B4 (VBUS), J1.B9 (VBUS), J2.4 (Pin_4)
Other:
- moved on the sheet: A10_USB_ID1, A11_USB_DM1, A12_USB_DP1, A9_USB_VBUS1, B2_BOOT1, NRST1, SOI8_SLCT1, U1, VBat1

Commit message: Fixed matrix LED wiring, shifted LED 0.2mm closer to switch. Changed capslock LED to addressable LED connected to matrix LED array.
Parts:
- removed CAPS1: LED, Keyboard_Parts_Footprint:LED_3020_REFLOW, symbol keyboard_parts:LED
- added CAPS_LED1: SK6812MINI-E_Rev, LED_SMD:LED_SK6812MINI-E_PLCC4_3.2x2.8mm_P1.5mm_1, symbol LED_SMD:SK6812MINI-E
- LED1: renamed from LED2; value SK6812MINI-E -> SK6812MINI-E_Rev
- LED10: renamed from LED11; value SK6812MINI-E -> SK6812MINI-E_Rev
- LED11: renamed from LED12; value SK6812MINI-E -> SK6812MINI-E_Rev
- LED12: renamed from LED13; value SK6812MINI-E -> SK6812MINI-E_Rev
- LED13: renamed from LED14; value SK6812MINI-E -> SK6812MINI-E_Rev
- LED14: renamed from LED15; value SK6812MINI-E -> SK6812MINI-E_Rev
- LED15: renamed from LED16; value SK6812MINI-E -> SK6812MINI-E_Rev
- LED16: renamed from LED17; value SK6812MINI-E -> SK6812MINI-E_Rev
- LED17: renamed from LED18; value SK6812MINI-E -> SK6812MINI-E_Rev
- LED18: renamed from LED19; value SK6812MINI-E -> SK6812MINI-E_Rev
- LED19: renamed from LED20; value SK6812MINI-E -> SK6812MINI-E_Rev
- LED2: renamed from LED3; value SK6812MINI-E -> SK6812MINI-E_Rev
- LED20: renamed from LED21; value SK6812MINI-E -> SK6812MINI-E_Rev
- LED21: renamed from LED22; value SK6812MINI-E -> SK6812MINI-E_Rev
- LED22: renamed from LED23; value SK6812MINI-E -> SK6812MINI-E_Rev
- LED23: renamed from LED24; value SK6812MINI-E -> SK6812MINI-E_Rev
- LED24: renamed from LED25; value SK6812MINI-E -> SK6812MINI-E_Rev
- LED25: renamed from LED26; value SK6812MINI-E -> SK6812MINI-E_Rev
- LED26: renamed from LED27; value SK6812MINI-E -> SK6812MINI-E_Rev
- LED27: renamed from LED28; value SK6812MINI-E -> SK6812MINI-E_Rev
- LED28: renamed from LED29; value SK6812MINI-E -> SK6812MINI-E_Rev
- LED29: renamed from LED30; value SK6812MINI-E -> SK6812MINI-E_Rev
- LED3: renamed from LED4; value SK6812MINI-E -> SK6812MINI-E_Rev
- LED30: renamed from LED31; value SK6812MINI-E -> SK6812MINI-E_Rev
- LED31: renamed from LED32; value SK6812MINI-E -> SK6812MINI-E_Rev
- LED32: renamed from LED33; value SK6812MINI-E -> SK6812MINI-E_Rev
- LED33: renamed from LED34; value SK6812MINI-E -> SK6812MINI-E_Rev
- LED34: renamed from LED35; value SK6812MINI-E -> SK6812MINI-E_Rev
- LED35: renamed from LED36; value SK6812MINI-E -> SK6812MINI-E_Rev
- LED36: renamed from LED37; value SK6812MINI-E -> SK6812MINI-E_Rev
- LED37: renamed from LED38; value SK6812MINI-E -> SK6812MINI-E_Rev
- LED38: renamed from LED39; value SK6812MINI-E -> SK6812MINI-E_Rev
- LED39: renamed from LED40; value SK6812MINI-E -> SK6812MINI-E_Rev
- LED4: renamed from LED5; value SK6812MINI-E -> SK6812MINI-E_Rev
- LED40: renamed from LED41; value SK6812MINI-E -> SK6812MINI-E_Rev
- LED41: renamed from LED42; value SK6812MINI-E -> SK6812MINI-E_Rev
- LED42: renamed from LED43; value SK6812MINI-E -> SK6812MINI-E_Rev
- LED43: renamed from LED44; value SK6812MINI-E -> SK6812MINI-E_Rev
- LED44: renamed from LED45; value SK6812MINI-E -> SK6812MINI-E_Rev
- LED45: renamed from LED46; value SK6812MINI-E -> SK6812MINI-E_Rev
- LED46: renamed from LED47; value SK6812MINI-E -> SK6812MINI-E_Rev
- LED47: renamed from LED48; value SK6812MINI-E -> SK6812MINI-E_Rev
- LED48: renamed from LED49; value SK6812MINI-E -> SK6812MINI-E_Rev
- LED49: renamed from LED50; value SK6812MINI-E -> SK6812MINI-E_Rev
- LED5: renamed from LED6; value SK6812MINI-E -> SK6812MINI-E_Rev
- LED50: renamed from LED51; value SK6812MINI-E -> SK6812MINI-E_Rev
- LED51: renamed from LED52; value SK6812MINI-E -> SK6812MINI-E_Rev
- LED52: renamed from LED53; value SK6812MINI-E -> SK6812MINI-E_Rev
- LED53: renamed from LED54; value SK6812MINI-E -> SK6812MINI-E_Rev
- LED54: renamed from LED55; value SK6812MINI-E -> SK6812MINI-E_Rev
- LED55: renamed from LED56; value SK6812MINI-E -> SK6812MINI-E_Rev
- LED56: renamed from LED57; value SK6812MINI-E -> SK6812MINI-E_Rev
- LED57: renamed from LED58; value SK6812MINI-E -> SK6812MINI-E_Rev
- LED58: renamed from LED59; value SK6812MINI-E -> SK6812MINI-E_Rev
- LED59: renamed from LED60; value SK6812MINI-E -> SK6812MINI-E_Rev
- LED6: renamed from LED7; value SK6812MINI-E -> SK6812MINI-E_Rev
- LED60: renamed from LED61; value SK6812MINI-E -> SK6812MINI-E_Rev
- LED61: renamed from LED62; value SK6812MINI-E -> SK6812MINI-E_Rev
- LED62: renamed from LED63; value SK6812MINI-E -> SK6812MINI-E_Rev
- LED63: renamed from LED64; value SK6812MINI-E -> SK6812MINI-E_Rev
- LED64: renamed from LED65; value SK6812MINI-E -> SK6812MINI-E_Rev
- LED65: renamed from LED66; value SK6812MINI-E -> SK6812MINI-E_Rev
- LED66: renamed from LED67; value SK6812MINI-E -> SK6812MINI-E_Rev
- LED67: renamed from LED68; value SK6812MINI-E -> SK6812MINI-E_Rev
- LED68: renamed from LED69; value SK6812MINI-E -> SK6812MINI-E_Rev
- LED69: renamed from LED70; value SK6812MINI-E -> SK6812MINI-E_Rev
- LED7: renamed from LED8; value SK6812MINI-E -> SK6812MINI-E_Rev
- LED70: renamed from LED71; value SK6812MINI-E -> SK6812MINI-E_Rev
- LED71: renamed from LED72; value SK6812MINI-E -> SK6812MINI-E_Rev
- LED72: renamed from LED73; value SK6812MINI-E -> SK6812MINI-E_Rev
- LED73: renamed from LED74; value SK6812MINI-E -> SK6812MINI-E_Rev
- LED74: renamed from LED75; value SK6812MINI-E -> SK6812MINI-E_Rev
- LED75: renamed from LED76; value SK6812MINI-E -> SK6812MINI-E_Rev
- LED76: renamed from LED77; value SK6812MINI-E -> SK6812MINI-E_Rev
- LED77: renamed from LED78; value SK6812MINI-E -> SK6812MINI-E_Rev
- LED78: renamed from LED79; value SK6812MINI-E -> SK6812MINI-E_Rev
- LED79: renamed from LED80; value SK6812MINI-E -> SK6812MINI-E_Rev
- LED8: renamed from LED9; value SK6812MINI-E -> SK6812MINI-E_Rev
- LED80: renamed from LED81; value SK6812MINI-E -> SK6812MINI-E_Rev
- LED81: renamed from LED82; value SK6812MINI-E -> SK6812MINI-E_Rev
- LED82: renamed from LED83; value SK6812MINI-E -> SK6812MINI-E_Rev
- LED83: renamed from LED84; value SK6812MINI-E -> SK6812MINI-E_Rev
- LED84: renamed from LED85; value SK6812MINI-E -> SK6812MINI-E_Rev
- LED9: renamed from LED10; value SK6812MINI-E -> SK6812MINI-E_Rev
- renumbered D1 to CAPS_D1, SW1 to CAPS_SW1, D2 to D1, D11 to D10, D12 to D11, D13 to D12, D14 to D13, D15 to D14, D16 to D15, D17 to D16, D18 to D17, D19 to D18, D20 to D19, D3 to D2, D21 to D20, D22 to D21, D23 to D22, D24 to D23, D25 to D24, D26 to D25, D27 to D26, D28 to D27, D29 to D28, D30 to D29, D4 to D3, D31 to D30, D32 to D31, D33 to D32, D34 to D33, D35 to D34, D36 to D35, D37 to D36, D38 to D37, D39 to D38, D40 to D39, D5 to D4, D41 to D40, D42 to D41, D43 to D42, D44 to D43, D45 to D44, D46 to D45, D47 to D46, D48 to D47, D49 to D48, D50 to D49, D6 to D5, D51 to D50, D52 to D51, D53 to D52, D54 to D53, D55 to D54, D56 to D55, D57 to D56, D58 to D57, D59 to D58, D60 to D59, D7 to D6, D61 to D60, D62 to D61, D63 to D62, D64 to D63, D65 to D64, D66 to D65, D67 to D66, D68 to D67, D69 to D68, D70 to D69, D8 to D7, D71 to D70, D72 to D71, D73 to D72, D74 to D73, D75 to D74, D76 to D75, D77 to D76, D78 to D77, D79 to D78, D80 to D79, D9 to D8, D81 to D80, D82 to D81, D83 to D82, D84 to D83, D85 to D84, D10 to D9, D86 to ESD1, SW2 to SW1, SW11 to SW10, SW12 to SW11, SW13 to SW12, SW14 to SW13, SW15 to SW14, SW16 to SW15, SW17 to SW16, SW18 to SW17, SW19 to SW18, SW20 to SW19, SW3 to SW2, SW21 to SW20, SW22 to SW21, SW23 to SW22, SW24 to SW23, SW25 to SW24, SW26 to SW25, SW27 to SW26, SW28 to SW27, SW29 to SW28, SW30 to SW29, SW4 to SW3, SW31 to SW30, SW32 to SW31, SW33 to SW32, SW34 to SW33, SW35 to SW34, SW36 to SW35, SW37 to SW36, SW38 to SW37, SW39 to SW38, SW40 to SW39, SW5 to SW4, SW41 to SW40, SW42 to SW41, SW43 to SW42, SW44 to SW43, SW45 to SW44, SW46 to SW45, SW47 to SW46, SW48 to SW47, SW49 to SW48, SW50 to SW49, SW6 to SW5, SW51 to SW50, SW52 to SW51, SW53 to SW52, SW54 to SW53, SW55 to SW54, SW56 to SW55, SW57 to SW56, SW58 to SW57, SW59 to SW58, SW60 to SW59, SW7 to SW6, SW61 to SW60, SW62 to SW61, SW63 to SW62, SW64 to SW63, SW65 to SW64, SW66 to SW65, SW67 to SW66, SW68 to SW67, SW69 to SW68, SW70 to SW69, SW8 to SW7, SW71 to SW70, SW72 to SW71, SW73 to SW72, SW74 to SW73, SW75 to SW74, SW76 to SW75, SW77 to SW76, SW78 to SW77, SW79 to SW78, SW80 to SW79, SW9 to SW8, SW81 to SW80, SW82 to SW81, SW83 to SW82, SW84 to SW83, SW85 to SW84, SW10 to SW9
Connections:
- net +5V: now also CAPS_LED1.1 (VDD)
- net GND: now also CAPS_LED1.4 (GND)
- net at LED47.3 (DIN): now also CAPS_LED1.2 (DOUT); no longer LED46.2 (DOUT)
- new net: CAPS_LED1.3 (DIN), LED46.2 (DOUT)
