File: Custom Keyboard Kicad/Custom Mechanical Keyboard.kicad_pcb (KiCad board)
At the start: 2 copper layers, 327 x 114.5 mm, 326 parts, among them J3 Conn_01x05, J4 Conn_01x06, J5 Conn_01x07, J6 Conn_01x20_Socket, J7 Conn_01x20_Socket, SW1 SW_SPST, SW10 SW_SPST, SW11 SW_SPST, SW12 SW_SPST, SW13 SW_SPST, SW14 SW_SPST, SW15 SW_SPST, SW16 SW_SPST, SW17 SW_SPST, SW18 SW_SPST, SW19 SW_SPST, SW2 SW_SPST, SW20 SW_SPST, SW21 SW_SPST, SW22 SW_SPST, SW23 SW_SPST, SW24 SW_SPST, SW25 SW_SPST, SW26 SW_SPST, SW27 SW_SPST, SW28 SW_SPST, SW29 SW_SPST, SW3 SW_SPST, SW30 SW_SPST, SW31 SW_SPST, SW32 SW_SPST, SW33 SW_SPST, SW34 SW_SPST, SW35 SW_SPST, SW36 SW_SPST, SW37 SW_SPST, SW38 SW_SPST, SW39 SW_SPST, SW4 SW_SPST, SW40 SW_SPST, SW41 SW_SPST, SW42 SW_SPST, SW43 SW_SPST, SW44 SW_SPST, SW45 SW_SPST, SW46 SW_SPST, SW47 SW_SPST, SW48 SW_SPST, SW49 SW_SPST, SW5 SW_SPST, SW50 SW_SPST, SW51 SW_SPST, SW52 SW_SPST, SW53 SW_SPST, SW54 SW_SPST, SW55 SW_SPST, SW56 SW_SPST, SW57 SW_SPST, SW58 SW_SPST, SW59 SW_SPST, SW6 SW_SPST, SW60 SW_SPST, SW61 SW_SPST, SW62 SW_SPST, SW63 SW_SPST, SW64 SW_SPST, SW65 SW_SPST, SW66 SW_SPST, SW67 SW_SPST, SW68 SW_SPST, SW69 SW_SPST, SW7 SW_SPST, SW70 SW_SPST, SW71 SW_SPST, SW72 SW_SPST, SW73 SW_SPST, SW74 SW_SPST, SW75 SW_SPST, SW76 SW_SPST, SW77 SW_SPST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

Commit message: Commit after exports
Parts:
- moved J5 2.00 mm to (49.0, 84.2)
- moved J3 0.50 mm to (53.0, 73.0)
- moved R3 0.50 mm to (58.5, 79.0)
- moved R4 0.50 mm to (61.0, 79.0)
- moved U3 0.50 mm to (53.8, 79.0)
- moved J4 0.27 mm to (50.1, 154.9)
Routing:
- net +5V: track 2143.8 -> 2146.4 mm
- net DIS_RST: track 71.9 -> 73.9 mm
- net DIS_DC: track 53.1 -> 55.1 mm
- net DIS_CS: track 55.1 -> 56.4 mm
- net DIS_SCK: track 61.5 -> 62.3 mm
- net DIS_MOSI: track 66.1 -> 66.9 mm
- net +3.3V: track 42.9 -> 43.6 mm
- net USB_DP: track 68.3 -> 67.8 mm
- net USB_DM: track 72.4 -> 71.9 mm
- net Net-(R3-Pad1): track 21.4 -> 20.9 mm
- net /Bat_Sense_IN: track 12.2 -> 11.7 mm
- net /5V_IN: track 13.5 -> 13.0 mm
- net GND: track 2171.0 -> 2170.8 mm, vias 14 -> 13
